File: design_files/ASL1001.sch (EAGLE design)
At the start: 4 parts

Commit message: update format
Other:
- note added: "3"
- note removed: "2"
Changed lines of the file:
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@@
 <text x="340.868" y="17.272" size="3.556" layer="94" font="vector">TinyLily LED - 0402</text>
 <text x="327.152" y="6.35" size="3.556" layer="94" font="vector">AS-SCH-ASL1001</text>
-<text x="416.56" y="6.858" size="3.556" layer="94" font="vector">2</text>
+<text x="416.56" y="6.858" size="3.556" layer="94" font="vector">3</text>
 <text x="45.72" y="35.56" size="3.048" layer="91">Released under the Creative Commons Attribution Share-Alike 3.0 License</text>
 <text x="45.72" y="30.48" size="3.048" layer="91">http://creativecommons.org/licenses/by-sa/3.0</text>
